File: v4/hardware/base_b/kicad/remote.sch (KiCad schematic (older format))
At the start: 29 parts, among them J12 Conn_01x04_Female, J16 Conn_01x04_Female, J19 Conn_01x03_Female, J20 Conn_01x04_Female, J5 Conn_01x03_Female, Q1 Q_NMOS_GDS, Q3 Q_NPN_EBC, SW1 SW_Push, SW2 SW_Push, SW4 SW_Push_Dual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

Commit message: update
Parts:
- removed gps1: Conn_01x04_Female, footprints:gps_neo6_blue_0, symbol Connector:Conn_01x04_Female
- removed sharp1: Conn_01x09_Female, footprints:Display_adafruit_sharp_13, symbol Connector:Conn_01x09_Female
- added AE1: Antenna_Shield, Connector_Coaxial:SMA_Amphenol_132289_EdgeMount, symbol device:Antenna_Shield
- added R7: 4.7K, Resistor_THT:R_Axial_DIN0309_L9.0mm_D3.2mm_P12.70mm_Horizontal, symbol Device:R
- added SW3: SW_Push, Button_Switch_THT:SW_Tactile_SPST_Angled_PTS645Vx58-2LFS, symbol Switch:SW_Push
- added U3: Adafruit_IMU_BNO005, footprints:IMU_Ada_BNO005, symbol dog:Adafruit_IMU_BNO005
- added U4: Adafruit_Sharp_Display_1_3, footprints:Display_adafruit_sharp_13, symbol dog:Adafruit_Sharp_Display_1_3
- added U5: neo-6m-black, footprints:gps_neo6m_black, symbol dog:neo-6m-black
- D2: symbol remote-rescue:DIODE-RocketScreamKicadLibrary -> remote-rescue:DIODE-RocketScreamKicadLibrary-remote-rescue
- SP1: symbol remote-rescue:SPEAKER_BUZZER5MM-Adafruit_Circuit_Playground-eagle-import -> remote-rescue:SPEAKER_BUZZER5MM-Adafruit_Circuit_Playground-eagle-import-remote-rescue
Connections:
- net labels added: A2, RX_D0, TX_D1
- net labels removed: DISP, EIN, EMD
- wire segments 33 -> 36
Other:
- note added: "Adafruit Sharp Display \n1.3""
- note added: "COMPASS"
- note added: "FEATHER"
- note added: "GPS NEO6M BLACK"
- note removed: "Adafruit Sharp"
- note removed: "GPS NEO6M BLUE"
- moved on the sheet: U1
Changed lines of the file:
@@
 Text GLabel 2700 4175 0    50   Input ~ 0
 A3
-Text Notes -3050 100  0    79   ~ 0
-Adafruit Sharp
+Text Notes -2050 -100 0    79   ~ 0
+Adafruit Sharp Display \n1.3"
 $Comp
 L Switch:SW_Push_Dual SW4
@@
 	1    0    0    -1
 $EndComp
-$Comp
-L Connector:Conn_01x09_Female sharp1
-U 1 1 61C52AE8
-P -2925 675
-F 0 "sharp1" V -2760 655 50  0000 C CNN
-F 1 "Conn_01x09_Female" V -2851 655 50  0000 C CNN
-F 2 "footprints:Display_adafruit_sharp_13" H -2925 675 50  0001 C CNN
-F 3 "~" H -2925 675 50  0001 C CNN
-	1    -2925 675
-	1    0    0    -1
-$EndComp
-Text GLabel -3125 575  0    50   Input ~ 0
+Text GLabel -1800 750  0    50   Input ~ 0
 SCK
-Text GLabel -3125 875  0    50   Input ~ 0
-EMD
-Text GLabel -3125 975  0    50   Input ~ 0
-DISP
-Text GLabel -3125 1075 0    50   Input ~ 0
-EIN
 $Comp
 L Device:R R6
@@
 	1350 3850 1125 3850
 Connection ~ 1350 3850
-Text GLabel -3125 775  0    50   Input ~ 0
+Text GLabel -1800 1050 0    50   Input ~ 0
 D5
-Text GLabel -3125 675  0    50   Input ~ 0
+Text GLabel -1800 900  0    50   Input ~ 0
 MOSI
 $Comp
@@
 	1    0    0    -1
 $EndComp
-Wire Wire Line
-	-3125 275  -3250 275
 $Comp
 L power:+3V3 #PWR0118
 U 1 1 61D9297E
-P -3250 275
-F 0 "#PWR0118" H -3250 125 50  0001 C CNN
-F 1 "+3V3" V -3235 403 50  0000 L CNN
-F 2 "" H -3250 275 50  0001 C CNN
-F 3 "" H -3250 275 50  0001 C CNN
-	1    -3250 275
+P -1800 300
+F 0 "#PWR0118" H -1800 150 50  0001 C CNN
+F 1 "+3V3" V -1785 428 50  0000 L CNN
+F 2 "" H -1800 300 50  0001 C CNN
+F 3 "" H -1800 300 50  0001 C CNN
+	1    -1800 300
 	1    0    0    -1
 $EndComp
@@
 L power:GND #PWR0114
 U 1 1 61C86AD2
-P -3550 500
-F 0 "#PWR0114" H -3550 250 50  0001 C CNN
-F 1 "GND" H -3545 327 50  0000 C CNN
-F 2 "" H -3550 500 50  0001 C CNN
-F 3 "" H -3550 500 50  0001 C CNN
-	1    -3550 500
-	1    0    0    -1
-$EndComp
-Wire Wire Line
-	-3125 475  -3550 475
-Wire Wire Line
-	-3550 475  -3550 500
+P -2200 600
+F 0 "#PWR0114" H -2200 350 50  0001 C CNN
+F 1 "GND" H -2195 427 50  0000 C CNN
+F 2 "" H -2200 600 50  0001 C CNN
+F 3 "" H -2200 600 50  0001 C CNN
+	1    -2200 600
+	1    0    0    -1
+$EndComp
 Wire Wire Line
 	2725 4075 2700 4075
@@
 $EndComp
 $Comp
-L remote-rescue:DIODE-RocketScreamKicadLibrary D2
+L remote-rescue:DIODE-RocketScreamKicadLibrary-remote-rescue D2
 U 1 1 61C856DC
 P -1300 6275
@@
 $EndComp
 $Comp
-L remote-rescue:SPEAKER_BUZZER5MM-Adafruit_Circuit_Playground-eagle-import SP1
+L remote-rescue:SPEAKER_BUZZER5MM-Adafruit_Circuit_Playground-eagle-import-remote-rescue SP1
 U 1 1 61C8B808
 P -1650 6275
@@
 Text GLabel -1025 4275 0    50   Input ~ 0
 A0
-$Comp
-L Connector:Conn_01x04_Female gps1
-U 1 1 61CE8D8B
-P 5050 1050
-F 0 "gps1" H 5078 1026 50  0000 L CNN
-F 1 "Conn_01x04_Female" H 5078 935 50  0000 L CNN
-F 2 "footprints:gps_neo6_blue_0" H 5050 1050 50  0001 C CNN
-F 3 "~" H 5050 1050 50  0001 C CNN
-	1    5050 1050
-	1    0    0    -1
-$EndComp
-Text Notes 4550 850  0    79   ~ 0
-GPS NEO6M BLUE
 Text GLabel 4150 4150 0    50   Input ~ 0
 EN
@@
 L mysensors_radios:RFM95HW U1
 U 1 1 61D2BB57
-P 3300 2200
-F 0 "U1" H 3300 2814 40  0000 C CNN
-F 1 "RFM95HW" H 3300 2738 40  0000 C CNN
-F 2 "footprints:RFM95" H 3300 2200 30  0001 C CIN
-F 3 "https://cdn-learn.adafruit.com/assets/assets/000/031/659/original/RFM95_96_97_98W.pdf?1460518717" H 3300 2647 60  0000 C CNN
-	1    3300 2200
+P 5450 -1050
+F 0 "U1" H 5450 -436 40  0000 C CNN
+F 1 "RFM95HW" H 5450 -512 40  0000 C CNN
+F 2 "footprints:RFM95" H 5450 -1050 30  0001 C CIN
+F 3 "https://cdn-learn.adafruit.com/assets/assets/000/031/659/original/RFM95_96_97_98W.pdf?1460518717" H 5450 -603 60  0000 C CNN
+	1    5450 -1050
 	1    0    0    -1
 $EndComp
@@
 	1    0    0    -1
 $EndComp
+$Comp
+L dog:Adafruit_IMU_BNO005 U3
+U 1 1 61D39165
+P 7350 1350
+F 0 "U3" H 7278 821 50  0000 L CNN
+F 1 "Adafruit_IMU_BNO005" H 7278 730 50  0000 L CNN
+F 2 "footprints:IMU_Ada_BNO005" H 7350 1350 50  0001 C CNN
+F 3 "" H 7350 1350 50  0001 C CNN
+	1    7350 1350
+	1    0    0    -1
+$EndComp
+$Comp
+L dog:Adafruit_Sharp_Display_1_3 U4
+U 1 1 61D40EC2
+P -1450 50
+F 0 "U4" H -1372 -754 50  0000 L CNN
+F 1 "Adafruit_Sharp_Display_1_3" H -1372 -845 50  0000 L CNN
+F 2 "footprints:Display_adafruit_sharp_13" H -1450 50  50  0001 C CNN
+F 3 "" H -1450 50  50  0001 C CNN
+	1    -1450 50
+	1    0    0    -1
+$EndComp
+Wire Wire Line
+	-1800 600  -2200 600
+Text GLabel -3750 2300 0    50   Input ~ 0
+A0
+Text GLabel -3750 3950 0    50   Input ~ 0
+DW
+Text GLabel -2850 2750 2    50   Input ~ 0
+D9
+Text GLabel -3750 2750 0    50   Input ~ 0
+A3
+Text GLabel -3750 3050 0    50   Input ~ 0
+A5
+Text GLabel -3750 2900 0    50   Input ~ 0
+A4
+Text GLabel -2850 3200 2    50   Input ~ 0
+SCL
+Text GLabel -2850 3350 2    50   Input ~ 0
+SDA
+$Comp
+L dog:neo-6m-black U5
+U 1 1 61D7113B
+P 2900 800
+F 0 "U5" H 3128 496 50  0000 L CNN
+F 1 "neo-6m-black" H 3128 405 50  0000 L CNN
+F 2 "footprints:gps_neo6m_black" H 2900 800 50  0001 C CNN
+F 3 "" H 2900 800 50  0001 C CNN
+	1    2900 800
+	1    0    0    -1
+$EndComp
+Text Notes 2450 700  0    79   ~ 0
+GPS NEO6M BLACK
+Text Notes 6650 1250 0    79   ~ 0
+COMPASS
+Text Notes -3900 1250 0    79   ~ 0
+FEATHER
+Text GLabel -3750 3650 0    50   Input ~ 0
+RX_D0
+Text GLabel -3750 3800 0    50   Input ~ 0
+TX_D1
+Text GLabel 2700 1050 0    50   Input ~ 0
+RX_D0
+Text GLabel 2700 1150 0    50   Input ~ 0
+TX_D1
+$Comp
+L power:+3V3 #PWR0101
+U 1 1 61D83F21
+P 2200 1350
+F 0 "#PWR0101" H 2200 1200 50  0001 C CNN
+F 1 "+3V3" V 2215 1478 50  0000 L CNN
+F 2 "" H 2200 1350 50  0001 C CNN
+F 3 "" H 2200 1350 50  0001 C CNN
+	1    2200 1350
+	1    0    0    -1
+$EndComp
+Wire Wire Line
+	2700 1350 2200 1350
+Wire Wire Line
+	2700 1250 2550 1250
+Wire Wire Line
+	2550 1250 2550 1450
+Text GLabel 6800 2000 0    50   Input ~ 0
+SCL
+Text GLabel 6800 2150 0    50   Input ~ 0
+SDA
+Text GLabel 2550 1450 0    50   Input ~ 0
+POWER_1
+$Comp
+L device:Antenna_Shield AE1
+U 1 1 61D92C44
+P 5250 -2000
+F 0 "AE1" H 5394 -1961 50  0000 L CNN
+F 1 "Antenna_Shield" H 5394 -2052 50  0000 L CNN
+F 2 "Connector_Coaxial:SMA_Amphenol_132289_EdgeMount" H 5250 -1900 50  0001 C CNN
+F 3 "" H 5250 -1900 50  0001 C CNN
+	1    5250 -2000
+	1    0    0    -1
+$EndComp
+$Comp
+L Device:R R7
+U 1 1 61DE7962
+P 3850 6975
+F 0 "R7" H 3920 7021 50  0000 L CNN
+F 1 "4.7K" H 3920 6930 50  0000 L CNN
+F 2 "Resistor_THT:R_Axial_DIN0309_L9.0mm_D3.2mm_P12.70mm_Horizontal" V 3780 6975 50  0001 C CNN
+F 3 "~" H 3850 6975 50  0001 C CNN
+	1    3850 6975
+	1    0    0    -1
+$EndComp
+$Comp
+L power:+3V3 #PWR0104
+U 1 1 61DE7C60
+P 3850 6825
+F 0 "#PWR0104" H 3850 6675 50  0001 C CNN
+F 1 "+3V3" H 3865 6998 50  0000 C CNN
+F 2 "" H 3850 6825 50  0001 C CNN
+F 3 "" H 3850 6825 50  0001 C CNN
+	1    3850 6825
+	1    0    0    -1
+$EndComp
+Text Notes 3950 6575 0    79   ~ 0
+BUTTON B
+$Comp
+L Switch:SW_Push SW3
+U 1 1 61DE7C6B
+P 4300 7125
+F 0 "SW3" H 4300 7410 50  0000 C CNN
+F 1 "SW_Push" H 4300 7319 50  0000 C CNN
+F 2 "Button_Switch_THT:SW_Tactile_SPST_Angled_PTS645Vx58-2LFS" H 4300 7325 50  0001 C CNN
+F 3 "~" H 4300 7325 50  0001 C CNN
+	1    4300 7125
+	1    0    0    -1
+$EndComp
+$Comp
+L power:GND #PWR0108
+U 1 1 61DE7C75
+P 4500 7125
+F 0 "#PWR0108" H 4500 6875 50  0001 C CNN
+F 1 "GND" H 4505 6952 50  0000 C CNN
+F 2 "" H 4500 7125 50  0001 C CNN
+F 3 "" H 4500 7125 50  0001 C CNN
+	1    4500 7125
+	1    0    0    -1
+$EndComp
+Wire Wire Line
+	4100 7125 3850 7125
+Text GLabel 3600 7125 0    50   Input ~ 0
+A2
+Wire Wire Line
+	3850 7125 3600 7125
+Connection ~ 3850 7125
 $EndSCHEMATC

Commit message: update
Parts:
- removed AE1: Antenna_Shield, Connector_Coaxial:SMA_Amphenol_132289_EdgeMount, symbol device:Antenna_Shield
- added J1: Conn_Coaxial, Connector_Coaxial:SMA_Amphenol_132134_Vertical, symbol Connector:Conn_Coaxial
Connections:
- net GND: now also J1.2 (Ext)
- net at U1.9 (ANA): now also J1.1 (In)
Changed lines of the file:
@@
 POWER_1
-$Comp
-L device:Antenna_Shield AE1
-U 1 1 61D92C44
-P 5250 -2000
-F 0 "AE1" H 5394 -1961 50  0000 L CNN
-F 1 "Antenna_Shield" H 5394 -2052 50  0000 L CNN
-F 2 "Connector_Coaxial:SMA_Amphenol_132289_EdgeMount" H 5250 -1900 50  0001 C CNN
-F 3 "" H 5250 -1900 50  0001 C CNN
-	1    5250 -2000
-	1    0    0    -1
-$EndComp
 $Comp
 L Device:R R7
@@
 	3850 7125 3600 7125
 Connection ~ 3850 7125
+$Comp
+L Connector:Conn_Coaxial J1
+U 1 1 61DED342
+P 4800 -2150
+F 0 "J1" H 4900 -2175 50  0000 L CNN
+F 1 "Conn_Coaxial" H 4900 -2266 50  0000 L CNN
+F 2 "Connector_Coaxial:SMA_Amphenol_132134_Vertical" H 4800 -2150 50  0001 C CNN
+F 3 " ~" H 4800 -2150 50  0001 C CNN
+	1    4800 -2150
+	1    0    0    -1
+$EndComp
+Wire Wire Line
+	4900 -1200 4600 -1200
+Wire Wire Line
+	4600 -1200 4600 -2150
+$Comp
+L power:GND #PWR0109
+U 1 1 61D58311
+P 4800 -1950
+F 0 "#PWR0109" H 4800 -2200 50  0001 C CNN
+F 1 "GND" H 4805 -2123 50  0000 C CNN
+F 2 "" H 4800 -1950 50  0001 C CNN
+F 3 "" H 4800 -1950 50  0001 C CNN
+	1    4800 -1950
+	1    0    0    -1
+$EndComp
 $EndSCHEMATC

Commit message: update
Parts:
- removed J12: Conn_01x04_Female, Connector_JST:JST_SH_SM04B-SRSS-TB_1x04-1MP_P1.00mm_Horizontal, symbol Connector:Conn_01x04_Female
- removed JP3: Jumper_NO_Small, Jumper:SolderJumper-2_P1.3mm_Open_Pad1.0x1.5mm, symbol Device:Jumper_NO_Small
- added J2: Conn_01x06_Female, Connector_PinHeader_2.54mm:PinHeader_1x06_P2.54mm_Vertical, symbol Connector:Conn_01x06_Female
- added J?: Conn_01x04_Female, Connector_JST:JST_SH_SM04B-SRSS-TB_1x04-1MP_P1.00mm_Horizontal, symbol Connector:Conn_01x04_Female
- added JP2: Jumper_NO_Small, Jumper:SolderJumper-2_P1.3mm_Open_Pad1.0x1.5mm, symbol device:Jumper_NO_Small
- Q1: footprint Package_TO_SOT_THT:TO-220-3_Vertical -> Package_TO_SOT_THT:TO-220-3_Horizontal_TabDown
Connections:
- net +3V3: now also U2.14 (3V3), J2.6 (Pin_6), J?.2 (Pin_2)
- net A0: now also U4.6 (CS); no longer R8.2
- net A2: now also R4.2, SW1.1, U2.19 (A2); no longer R7.2, SW3.1
- net A3: now also R3.2, SW2.1; no longer J19.3 (Pin_3)
- net A4: now also R7.2, SW3.1; no longer R4.2, SW1.1
- net A5: now also J19.3 (Pin_3); no longer R3.2, SW2.1
- net D5: now also U1.5 (NSS), U2.10 (D5); no longer U4.6 (CS)
- net D9: now also U1.14 (DIO0)
- net EN: now also U2.2 (EN)
- net GND: now also U2.16 (GND), J2.1 (Pin_1), J?.1 (Pin_1)
- net MOSI: now also U1.3 (MOSI), U2.24 (MOSI)
- net SCK: now also U1.4 (SCK), U2.23 (SCK)
- net SCL: now also J?.4 (Pin_4)
- net SDA: now also J?.3 (Pin_3)
- net ~RESET: now also U2.13 (~RESET)
- net at U1.15 (DIO1): now also JP2.1
- net MISO: now reaches U1.2 (MISO)
- net MISO: now also U2.25 (MISO)
- net D6: now reaches U1.6 (RESET)
- net D6: now also U2.9 (D6)
- net VBAT: now reaches U2.1 (VBAT)
- net AREF: now reaches U2.15 (AREF)
- net A1: now reaches U2.18 (A1)
- net A1: now also R8.2, J2.5 (Pin_5)
- net VBUS: now reaches U2.3 (VBUS)
- net D13: now reaches U2.4 (D13)
- net D13: now also J2.4 (Pin_4)
- net D12: now reaches U2.5 (D12)
- net D12: now also J2.3 (Pin_3)
- net D11: now reaches U2.6 (D11)
- net D11: now also J2.2 (Pin_2)
- net D10: now reaches U2.7 (D10)
- net D10: now also JP2.2
Other:
- note added: "BUTTON C"
- note added: "i2c breakout"
- note removed: "LORA"
- moved on the sheet: D2, H1, H2, H5, H6, J1, J16, J19, J20, J5, JP1, Q1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

Commit message: nice board layout for v4 base_b
Parts:
- removed R5: R, Resistor_THT:R_Axial_DIN0309_L9.0mm_D3.2mm_P12.70mm_Horizontal, symbol Device:R
- gave numbers to parts that had none: 1
- renumbered D2 to D1, R6 to R3, R7 to R4, R3 to R5, R4 to R6, R8 to R7
Connections:
- net +3V3: now also U3.1 (VIN)
- net GND: now also J19.2 (Pin_2), U3.3 (GND)
Other:
- moved on the sheet: J19
Changed lines of the file:
@@
 i2c pullups
 $Comp
-L Device:R R3
+L Device:R R5
 U 1 1 6028DEF2
 P 6650 2575
-F 0 "R3" H 6720 2621 50  0000 L CNN
+F 0 "R5" H 6720 2621 50  0000 L CNN
 F 1 "4.7K" H 6720 2530 50  0000 L CNN
 F 2 "Resistor_THT:R_Axial_DIN0309_L9.0mm_D3.2mm_P12.70mm_Horizontal" V 6580 2575 50  0001 C CNN
@@
 BUTTON A
 $Comp
-L Device:R R4
+L Device:R R6
 U 1 1 60FBA6C0
 P 6575 1300
-F 0 "R4" H 6645 1346 50  0000 L CNN
+F 0 "R6" H 6645 1346 50  0000 L CNN
 F 1 "4.7K" H 6645 1255 50  0000 L CNN
 F 2 "Resistor_THT:R_Axial_DIN0309_L9.0mm_D3.2mm_P12.70mm_Horizontal" V 6505 1300 50  0001 C CNN
@@
 L power:GND #PWR0107
 U 1 1 6193871C
-P 3925 7425
-F 0 "#PWR0107" H 3925 7175 50  0001 C CNN
-F 1 "GND" H 3930 7252 50  0000 C CNN
-F 2 "" H 3925 7425 50  0001 C CNN
-F 3 "" H 3925 7425 50  0001 C CNN
-	1    3925 7425
-	1    0    0    -1
-$EndComp
-$Comp
-L Device:R R5
-U 1 1 6193A6F6
-P 3925 7275
-F 0 "R5" H 3995 7321 50  0000 L CNN
-F 1 "R" H 3995 7230 50  0000 L CNN
-F 2 "Resistor_THT:R_Axial_DIN0309_L9.0mm_D3.2mm_P12.70mm_Horizontal" V 3855 7275 50  0001 C CNN
-F 3 "~" H 3925 7275 50  0001 C CNN
-	1    3925 7275
-	1    0    0    -1
-$EndComp
-$Comp
-L Connector:Conn_01x03_Female J19
-U 1 1 61938716
-P 4450 7125
-F 0 "J19" H 4478 7151 50  0000 L CNN
-F 1 "Conn_01x03_Female" H 4478 7060 50  0000 L CNN
-F 2 "Connector_PinSocket_2.54mm:PinSocket_1x03_P2.54mm_Vertical" H 4450 7125 50  0001 C CNN
-F 3 "~" H 4450 7125 50  0001 C CNN
-	1    4450 7125
+P 3950 7100
+F 0 "#PWR0107" H 3950 6850 50  0001 C CNN
+F 1 "GND" H 3955 6927 50  0000 C CNN
+F 2 "" H 3950 7100 50  0001 C CNN
+F 3 "" H 3950 7100 50  0001 C CNN
+	1    3950 7100
 	1    0    0    -1
 $EndComp
 Text Notes 4100 6875 0    79   ~ 0
 Write Permit\n
-Text GLabel 4250 7225 0    50   Input ~ 0
+Text GLabel 4350 7200 0    50   Input ~ 0
 A5
 Text Notes 1100 2350 0    79   ~ 0
@@
 SCK
 $Comp
-L Device:R R6
+L Device:R R3
 U 1 1 61C43F0B
 P 5100 5000
-F 0 "R6" H 5170 5046 50  0000 L CNN
+F 0 "R3" H 5170 5046 50  0000 L CNN
 F 1 "10K" H 5170 4955 50  0000 L CNN
 F 2 "Resistor_THT:R_Axial_DIN0309_L9.0mm_D3.2mm_P12.70mm_Horizontal" V 5030 5000 50  0001 C CNN
@@
 	1    0    0    -1
 $EndComp
-Wire Wire Line
-	4275 7125 4250 7125
-Connection ~ 4250 7125
-Wire Wire Line
-	4250 7125 3925 7125
 $Comp
 L Device:Q_NPN_EBC Q3
@@
 $EndComp
 $Comp
-L remote-rescue:DIODE-RocketScreamKicadLibrary-remote-rescue D2
+L remote-rescue:DIODE-RocketScreamKicadLibrary-remote-rescue D1
 U 1 1 61C856DC
 P 3850 5525
-F 0 "D2" V 3804 5603 50  0000 L CNN
+F 0 "D1" V 3804 5603 50  0000 L CNN
 F 1 "DIODE" V 3895 5603 50  0000 L CNN
 F 2 "Diode_THT:D_5W_P12.70mm_Horizontal" H 3850 5325 60  0001 C CNN
@@
 $EndComp
 $Comp
-L Device:R R8
+L Device:R R7
 U 1 1 61C856E2
 P 3050 5925
-F 0 "R8" V 2843 5925 50  0000 C CNN
+F 0 "R7" V 2843 5925 50  0000 C CNN
 F 1 "R" V 2934 5925 50  0000 C CNN
 F 2 "Resistor_THT:R_Axial_DIN0309_L9.0mm_D3.2mm_P12.70mm_Horizontal" V 2980 5925 50  0001 C CNN
@@
 POWER_1
 $Comp
-L Device:R R7
+L Device:R R4
 U 1 1 61DE7962
 P 6700 3775
-F 0 "R7" H 6770 3821 50  0000 L CNN
+F 0 "R4" H 6770 3821 50  0000 L CNN
 F 1 "4.7K" H 6770 3730 50  0000 L CNN
 F 2 "Resistor_THT:R_Axial_DIN0309_L9.0mm_D3.2mm_P12.70mm_Horizontal" V 6630 3775 50  0001 C CNN
@@
 QWIIC
 $Comp
-L Connector:Conn_01x04_Female J?
+L Connector:Conn_01x04_Female J3
 U 1 1 61F816B3
 P 9000 5125
-F 0 "J?" H 9028 5101 50  0000 L CNN
+F 0 "J3" H 9028 5101 50  0000 L CNN
 F 1 "Conn_01x04_Female" V 9175 4675 50  0000 L CNN
 F 2 "Connector_JST:JST_SH_SM04B-SRSS-TB_1x04-1MP_P1.00mm_Horizontal" H 9000 5125 50  0001 C CNN
@@
 SDA
 $Comp
-L power:+3V3 #PWR?
+L power:+3V3 #PWR0120
 U 1 1 61F816C1
 P 8625 5125
-F 0 "#PWR?" H 8625 4975 50  0001 C CNN
+F 0 "#PWR0120" H 8625 4975 50  0001 C CNN
 F 1 "+3V3" H 8640 5298 50  0000 C CNN
 F 2 "" H 8625 5125 50  0001 C CNN
@@
 $EndComp
 $Comp
-L power:GND #PWR?
+L power:GND #PWR0121
 U 1 1 61F816CB
 P 8400 5025
-F 0 "#PWR?" H 8400 4775 50  0001 C CNN
+F 0 "#PWR0121" H 8400 4775 50  0001 C CNN
 F 1 "GND" H 8405 4852 50  0000 C CNN
 F 2 "" H 8400 5025 50  0001 C CNN
@@
 	1    0    0    -1
 $EndComp
+$Comp
+L power:GND #PWR0122
+U 1 1 6201B316
+P 8600 1500
+F 0 "#PWR0122" H 8600 1250 50  0001 C CNN
+F 1 "GND" H 8605 1327 50  0000 C CNN
+F 2 "" H 8600 1500 50  0001 C CNN
+F 3 "" H 8600 1500 50  0001 C CNN
+	1    8600 1500
+	1    0    0    -1
+$EndComp
+$Comp
+L power:+3V3 #PWR0123
+U 1 1 6201B81A
+P 8600 1200
+F 0 "#PWR0123" H 8600 1050 50  0001 C CNN
+F 1 "+3V3" H 8615 1373 50  0000 C CNN
+F 2 "" H 8600 1200 50  0001 C CNN
+F 3 "" H 8600 1200 50  0001 C CNN
+	1    8600 1200
+	1    0    0    -1
+$EndComp
+Wire Wire Line
+	8950 1200 8600 1200
+Wire Wire Line
+	8950 1500 8600 1500
+$Comp
+L Connector:Conn_01x03_Female J19
+U 1 1 61938716
+P 4550 7100
+F 0 "J19" H 4578 7126 50  0000 L CNN
+F 1 "Conn_01x03_Female" H 4578 7035 50  0000 L CNN
+F 2 "Connector_PinSocket_2.54mm:PinSocket_1x03_P2.54mm_Vertical" H 4550 7100 50  0001 C CNN
+F 3 "~" H 4550 7100 50  0001 C CNN
+	1    4550 7100
+	1    0    0    -1
+$EndComp
+Wire Wire Line
+	4350 7100 3950 7100
 $EndSCHEMATC

Commit message: update
Parts:
- Q1: footprint Package_TO_SOT_THT:TO-220-3_Horizontal_TabDown -> Package_TO_SOT_THT:TO-220-3_Horizontal_TabUp
Changed lines of the file:
@@
 F 0 "Q1" H 5504 4896 50  0000 L CNN
 F 1 "Q_NMOS_GDS" H 5504 4805 50  0000 L CNN
-F 2 "Package_TO_SOT_THT:TO-220-3_Horizontal_TabDown" H 5500 4950 50  0001 C CNN
+F 2 "Package_TO_SOT_THT:TO-220-3_Horizontal_TabUp" H 5500 4950 50  0001 C CNN
 F 3 "~" H 5300 4850 50  0001 C CNN
 	1    5300 4850
