File: v4/hardware/base_b/kicad/remote.kicad_pcb (KiCad board)
At the start: 2 copper layers, 53.3 x 115.3 mm, 32 parts, among them J1 Conn_Coaxial, J16 Conn_01x04_Female, J19 Conn_01x03_Female, J2 Conn_01x06_Female, J20 Conn_01x04_Female, J5 Conn_01x03_Female, Q1 Q_NMOS_GDS, Q3 Q_NPN_EBC, SW1 SW_Push, SW2 SW_Push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

Commit message: fully routed power lines
Routing:
- net GND: track 386.9 -> 405.0 mm
- net +3V3: track 253.9 -> 270.3 mm, vias 16 -> 18
Changed lines of the file:
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@@
     (thickness 1.6)
     (drawings 79)
-    (tracks 181)
+    (tracks 190)
     (zones 0)
     (modules 32)
@@
   (segment (start 15.33538 13.7705) (end 15.33538 32.02462) (width 0.7) (layer B.Cu) (net 1))
   (segment (start 15.33538 32.02462) (end 15.33538 33.61462) (width 0.7) (layer B.Cu) (net 1))
+  (segment (start 6.25 55.74) (end 6.3 55.69) (width 0.7) (layer F.Cu) (net 1))
+  (segment (start -11.72 55.74) (end 6.25 55.74) (width 0.7) (layer F.Cu) (net 1))
   (segment (start -7.607136 63.98192) (end -3.549668 63.98192) (width 0.7) (layer F.Cu) (net 2))
   (segment (start -3.549668 63.98192) (end 0.5078 63.98192) (width 0.7) (layer F.Cu) (net 2))
@@
   (segment (start -5.08 27.99) (end -5.16 27.91) (width 0.7) (layer B.Cu) (net 2))
   (segment (start -25.79 27.91) (end -26.07 27.63) (width 0.7) (layer F.Cu) (net 2))
-  (segment (start -5.16 27.91) (end -25.79 27.91) (width 0.7) (layer F.Cu) (net 2))
   (via (at -23.67 -7.33) (size 0.8) (drill 0.4) (layers F.Cu B.Cu) (net 2))
   (segment (start -23.72106 1.96088) (end -23.72106 -7.27894) (width 0.7) (layer B.Cu) (net 2))
@@
   (segment (start -11.88 11.5) (end -11.81 11.57) (width 0.7) (layer B.Cu) (net 2))
   (via (at -23.17 11.57) (size 0.8) (drill 0.4) (layers F.Cu B.Cu) (net 2))
-  (segment (start -11.81 11.57) (end -23.17 11.57) (width 0.7) (layer F.Cu) (net 2))
   (segment (start -23.17 2.51194) (end -23.72106 1.96088) (width 0.7) (layer B.Cu) (net 2))
   (segment (start -23.17 11.57) (end -23.17 2.51194) (width 0.7) (layer B.Cu) (net 2))
@@
   (segment (start -17.5756 -7.22) (end -17.70942 -7.35382) (width 0.7) (layer F.Cu) (net 2))
   (segment (start -11.27 -7.22) (end -17.5756 -7.22) (width 0.7) (layer F.Cu) (net 2))
+  (via (at -17.77 11.57) (size 0.8) (drill 0.4) (layers F.Cu B.Cu) (net 2))
+  (segment (start -17.78 11.57) (end -17.77 11.57) (width 0.7) (layer F.Cu) (net 2))
+  (segment (start -17.78 11.57) (end -23.17 11.57) (width 0.7) (layer F.Cu) (net 2))
+  (segment (start -11.81 11.57) (end -17.78 11.57) (width 0.7) (layer F.Cu) (net 2))
+  (via (at -17.89 27.91) (size 0.8) (drill 0.4) (layers F.Cu B.Cu) (net 2))
+  (segment (start -17.77 27.79) (end -17.89 27.91) (width 0.7) (layer B.Cu) (net 2))
+  (segment (start -17.77 11.57) (end -17.77 27.79) (width 0.7) (layer B.Cu) (net 2))
+  (segment (start -5.16 27.91) (end -17.89 27.91) (width 0.7) (layer F.Cu) (net 2))
+  (segment (start -17.89 27.91) (end -25.79 27.91) (width 0.7) (layer F.Cu) (net 2))
 )

Commit message: update
Parts:
- moved H1 0.46 mm to (-28.1, 71.9)
- moved H5 0.05 mm to (17.8, -21.8)
Routing:
- net SDA: track 0.00 -> 189.5 mm, vias 0 -> 11
- net Net-(D1-Pad2): track 0.00 -> 173.8 mm, vias 0 -> 10
- net SCL: track 0.00 -> 141.8 mm, vias 0 -> 9
- net D10: track 0.00 -> 119.4 mm, vias 0 -> 4
- net D13: track 0.00 -> 118.1 mm, vias 0 -> 5
- net D6: track 0.00 -> 105.8 mm, vias 0 -> 5
- net D9: track 0.00 -> 91.8 mm, vias 0 -> 6
- net D12: track 0.00 -> 90.7 mm, vias 0 -> 3
- net D11: track 0.00 -> 89.1 mm, vias 0 -> 5
- net A1: track 0.00 -> 85.6 mm, vias 0 -> 3
- net A2: track 0.00 -> 84.0 mm, vias 0 -> 5
- net A0: track 0.00 -> 80.1 mm, vias 0 -> 2
- net SCK: track 0.00 -> 78.0 mm, vias 0 -> 5
- net A3: track 0.00 -> 69.3 mm, vias 0 -> 2
- net MOSI: track 0.00 -> 69.3 mm, vias 0 -> 6
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Other:
- board text added: "pvos.org/tracker"
- board text added: "tracker"
- board text added: "tracker v0.1"
- board text added: "v0.1"
