File: tracker_v_0.1/hardware/base/kicad/remote.kicad_sch (KiCad schematic)
At the start: 31 parts, among them J12 Conn_01x04_Female, J15 Conn_01x09_Female, J19 Conn_01x03_Female, J2 Conn_01x12_Female, J20 Conn_01x04_Female, J3 Conn_01x16_Female, J4 Conn_01x06_Female, J5 Conn_01x03_Female, J6 Conn_01x05_Female, Q1 Q_NMOS_GDS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

Commit message: reorg
Parts:
- removed H1, H2, H5, H6: MountingHole_Pad, MountingHole:MountingHole_2.7mm_M2.5_Pad, symbol Mechanical:MountingHole_Pad
- added H10, H11, H12, H3, H4, H7, H8, H9: MountingHole, footprints:MOUNTINGHOLE_2.5_PLATED, symbol Mechanical:MountingHole
