File: tracker_v_0.1/hardware/base/kicad/remote.sch (KiCad schematic (older format))
At the start: 40 parts, among them J1 Conn_01x02_Female, J10 Conn_01x16_Female, J11 Conn_01x10_Female, J12 Conn_01x04_Female, J14 Conn_01x08_Female, J15 Conn_01x09_Female, J16 Conn_01x04_Female, J17 Conn_01x07_Female, J19 Conn_01x03_Female, J2 Conn_01x12_Female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

Commit message: reorg
Parts:
- removed C1: 10uF, Capacitor_THT:CP_Radial_D5.0mm_P2.50mm, symbol device:C
- removed C2: 22uF, Capacitor_THT:CP_Radial_D5.0mm_P2.50mm, symbol device:C
- removed D1: D, Diode_THT:D_5W_P12.70mm_Horizontal, symbol Device:D
- removed J1: Conn_01x02_Female, Connector_JST:JST_PH_S2B-PH-K_1x02_P2.00mm_Horizontal, symbol Connector:Conn_01x02_Female
- removed J10, J3: Conn_01x16_Female, Connector_PinSocket_2.54mm:PinSocket_1x16_P2.54mm_Vertical, symbol Connector:Conn_01x16_Female
- removed J11: Conn_01x10_Female, Connector_PinSocket_2.54mm:PinSocket_1x10_P2.54mm_Vertical, symbol Connector:Conn_01x10_Female
- removed J12: Conn_01x04_Female, Connector_JST:JST_SH_SM04B-SRSS-TB_1x04-1MP_P1.00mm_Horizontal, symbol Connector:Conn_01x04_Female
- removed J14: Conn_01x08_Female, Connector_PinSocket_2.54mm:PinSocket_1x08_P2.54mm_Vertical, symbol Connector:Conn_01x08_Female
- removed J15: Conn_01x09_Female, Connector_PinSocket_2.54mm:PinSocket_1x09_P2.54mm_Vertical, symbol Connector:Conn_01x09_Female
- removed J17: Conn_01x07_Female, Connector_PinSocket_2.54mm:PinSocket_1x07_P2.54mm_Vertical, symbol Connector:Conn_01x07_Female
- removed J2, J9: Conn_01x12_Female, Connector_PinSocket_2.54mm:PinSocket_1x12_P2.54mm_Vertical, symbol Connector:Conn_01x12_Female
- removed J4: Conn_01x03_Female, Connector_PinSocket_2.54mm:PinSocket_1x03_P2.54mm_Vertical, symbol Connector:Conn_01x03_Female
- removed J7: Barrel_Jack_MountingPin, Connector_BarrelJack:BarrelJack_Horizontal, symbol Connector:Barrel_Jack_MountingPin
- removed J8: Screw_Terminal_01x02, TerminalBlock_Phoenix:TerminalBlock_Phoenix_PT-1,5-2-5.0-H_1x02_P5.00mm_Horizontal, symbol Connector:Screw_Terminal_01x02
- removed JP3: Jumper_NO_Small, Jumper:SolderJumper-2_P1.3mm_Open_Pad1.0x1.5mm, symbol Device:Jumper_NO_Small
- removed R5: R, Resistor_THT:R_Axial_DIN0309_L9.0mm_D3.2mm_P12.70mm_Horizontal, symbol Device:R
- added J1: Conn_Coaxial, Connector_Coaxial:SMA_Amphenol_132134_Vertical, symbol Connector:Conn_Coaxial
- added J2: Conn_01x06_Female, Connector_PinHeader_2.54mm:PinHeader_1x06_P2.54mm_Vertical, symbol Connector:Conn_01x06_Female
- added JP2: Jumper_NO_Small, Jumper:SolderJumper-2_P1.3mm_Open_Pad1.0x1.5mm, symbol device:Jumper_NO_Small
- added R4: 4.7K, Resistor_THT:R_Axial_DIN0309_L9.0mm_D3.2mm_P12.70mm_Horizontal, symbol Device:R
- added SW3: SW_Push, Button_Switch_THT:SW_Tactile_SPST_Angled_PTS645Vx58-2LFS, symbol Switch:SW_Push
- added U1: RFM95HW, footprints:RFM95, symbol mysensors_radios:RFM95HW
- added U2: feather, footprints:feather, symbol dog:feather
- added U3: Adafruit_IMU_BNO005, footprints:IMU_Ada_BNO005, symbol dog:Adafruit_IMU_BNO005
- added U4: Adafruit_Sharp_Display_1_3, footprints:Display_adafruit_sharp_13, symbol dog:Adafruit_Sharp_Display_1_3
- added U5: neo-6m-black, footprints:gps_neo6m_black, symbol dog:neo-6m-black
- D1: renamed from D2; symbol RocketScreamKicadLibrary:DIODE -> remote-rescue:DIODE-RocketScreamKicadLibrary-remote-rescue
- Q1: footprint Package_TO_SOT_THT:TO-220-3_Vertical -> Package_TO_SOT_THT:TO-220-3_Horizontal_TabUp
- SP1: symbol remote-rescue:SPEAKER_BUZZER5MM-Adafruit_Circuit_Playground-eagle-import -> remote-rescue:SPEAKER_BUZZER5MM-Adafruit_Circuit_Playground-eagle-import-remote-rescue
- renumbered R6 to R3, R3 to R5, R4 to R6, R8 to R7
Connections:
- net VBAT_EXT is gone; now on net GND: J5.3 (Pin_3)
- net +3V3: now also J2.6 (Pin_6), R4.1, U1.13 (3.3V), U2.14 (3V3), U3.1 (VIN), U4.1 (VIN), U5.5 (VCC)
- net A0: now also J2.5 (Pin_5), JP2.2, U2.17 (A0); no longer R7.2
- net A1: now also R7.2, J2.4 (Pin_4), U2.18 (A1)
- net A2: now also R6.2, SW1.1, U2.19 (A2)
- net A3: now also R5.2, SW2.1, U2.20 (A3); no longer J19.3 (Pin_3)
- net A4: now also R4.2, SW3.1, U2.21 (A4); no longer R6.2, SW1.1
- net A5: now also J19.3 (Pin_3), U2.22 (A5); no longer R5.2, SW2.1
- net AREF: now also U2.15 (AREF)
- net D10: now also J2.2 (Pin_2), U2.7 (D10)
- net D11: now also U1.5 (NSS), U2.6 (D11)
- net D12: now also U1.14 (DIO0), U2.5 (D12)
- net D13: now also J2.3 (Pin_3), U2.4 (D13)
- net D5: now also U2.10 (D5), U4.6 (CS)
- net D6: now also U1.6 (RESET), U2.9 (D6)
- net D9: now also U2.8 (D9)
- net DW: now also U2.28 (WC)
- net EN: now also J5.2 (Pin_2), U2.2 (EN)
- net GND: now also J19.2 (Pin_2), J1.2 (Ext), J2.1 (Pin_1), SW3.2, U1.1 (GND), U1.10 (GND), U1.8 (GND), U2.16 (GND), U3.3 (GND), U4.3 (GND); no longer J5.1 (Pin_1)
- net MISO: now also U1.2 (MISO), U2.25 (MISO)
- net MOSI: now also U1.3 (MOSI), U2.24 (MOSI), U4.5 (DI)
- net POWER_1: now also U5.4 (GND)
- net RX_D0: now also U2.26 (RX_D0), U5.2 (TXD)
- net SCK: now also U1.4 (SCK), U2.23 (SCK), U4.4 (CLK)
- net SCL: now also U2.11 (SCL), U3.4 (SCL)
- net SDA: now also U2.12 (SDA), U3.5 (SDA)
- net TX_D1: now also U2.27 (TX_D1), U5.3 (RXD)
- net VBAT: now also U2.1 (VBAT); no longer J5.2 (Pin_2)
- net VBUS: now also U2.3 (VBUS)
- net ~RESET: now also U2.13 (~RESET)
- new net: JP2.1, U1.15 (DIO1)
- new net: J1.1 (In), U1.9 (ANA)
Other:
- note added: "Adafruit Sharp Display \n1.3""
- note added: "BUTTON C"
- note added: "COMPASS"
- note added: "FEATHER"
- note added: "GPS NEO6M BLACK"
- note added: "i2c breakout / optional oled display"
- note removed: "'Air baffle' headers for SCD30"
- note removed: "5V DC-DC"
- note removed: "Adafruit 128x128"
- note removed: "Adafruit Sharp"
- note removed: "Airlift Featherwing"
- note removed: "Feather"
- note removed: "JST VBat Lithium Ion"
- note removed: "LORA"
- note removed: "POWER"
- note removed: "SCD30"
- note removed: "SCD30 is switched by Q1;\nalternatively, solder jumper\n"
- note removed: "by default, D13, D12, D11, \nand D10 are all used by \nesp32 featherwing"
- note removed: "pin 9 was D7; is now D6\npin 10 was D5; is now D2"
- moved on the sheet: D1, H1, H2, H5, H6, J16, J19, J20, J5, JP1, Q1, Q3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
