File: tracker_v_0.1/hardware/node/kicad/remote.kicad_pcb (KiCad board)
At the start: 2 copper layers, 29.5 x 69.4 mm, 13 parts, among them J1 Conn_Coaxial, J19 Conn_01x03_Female, J20 Conn_01x04_Female, J5 Conn_01x03_Female, Q1 Q_NMOS_GDS, U1 RFM95HW, U2 feather, U5 neo-6m-black

Commit message: fully routed node
Parts:
- removed JP2: Jumper_NO_Small, Jumper:SolderJumper-2_P1.3mm_Open_Pad1.0x1.5mm
- added J2: Conn_01x05_Female, Connector_PinSocket_2.54mm:PinSocket_1x05_P2.54mm_Vertical, F.Cu at (23.6, 125.4)
- moved J19 0.57 mm to (23.6, 109.7)
- moved J5 0.44 mm to (23.6, 131.7)
- turned JP1 to 270 degrees
- renumbered R2 to R1, R1 to R2
Connections:
- Q1 pad 1: D9 -> A4
- R3 pad 1: D9 -> A4
- U1 pad 14: D12 -> D9
- U1 pad 15: Net-(JP2-Pad1) -> A3
- U1 pad 5: D11 -> D5
- U2 pad 10: (no net) -> D5
- U2 pad 18: (no net) -> A1
- U2 pad 19: (no net) -> A2
- U2 pad 20: (no net) -> A3
- U2 pad 21: (no net) -> A4
- U2 pad 5: D12 -> (no net)
- U2 pad 6: D11 -> (no net)
Routing:
- net GND: track 0.00 -> 160.9 mm, vias 0 -> 9
- net +3V3: track 0.00 -> 97.9 mm, vias 0 -> 10
- net A2: track 0.00 -> 61.1 mm, vias 0 -> 2
- net SCL: track 0.00 -> 58.8 mm, vias 0 -> 2
- net SDA: track 0.00 -> 54.8 mm, vias 0 -> 3
- net A5: track 0.00 -> 46.9 mm, vias 0 -> 4
- net A3: track 0.00 -> 45.8 mm, vias 0 -> 3
- net A1: track 0.00 -> 41.4 mm, vias 0 -> 6
- net A0: track 0.00 -> 40.3 mm, vias 0 -> 2
- net A4: track 0.00 -> 40.1 mm, vias 0 -> 3
- net POWER_1: track 0.00 -> 40.0 mm, vias 0 -> 4
- net TX_D1: track 0.00 -> 30.9 mm, vias 0 -> 3
- net D9: track 0.00 -> 28.0 mm, vias 0 -> 2
- net SCK: track 0.00 -> 26.7 mm, vias 0 -> 3
- net D6: track 0.00 -> 23.9 mm, vias 0 -> 3
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Other:
- board text added: "1"
- board text added: "16"
- board text added: "3V"
- board text added: "8"
- board text added: "A0"
- board text added: "A1"
- board text added: "A2"
- board text added: "A4"
- board text added: "ANT"
- board text added: "G"
- board text added: "G1"
- board text added: "GND"
- board text added: "LOG"
- board text added: "OFF"
- board text added: "ON"
- board text added: "PROG"
- board text added: "RX_D1"
- board text added: "TX_D1"
- board text added: "node"
- board text added: "pvos.org/node"
- board text added: "v0.1"
